File: shield/Shield_Galileo.sch (KiCad schematic (older format))
At the start: 20 parts, among them J1 Connector_Encoder, J2 End_Sensor, J3 27V Power Supply, J4 Motor, U1 LS7366R, U2 Intel_Galileo_Gen2, U3 L298HN, U4 74HC04, Y1 32MHz

Commit message: Add new Shield files
Parts:
- J1: symbol Quanser_2DSFJE_Library:Connector_Encoder -> Shield_Galileo-rescue:Connector_Encoder-Quanser_2DSFJE_Library
- J2: symbol Quanser_2DSFJE_Library:End_Sensor -> Shield_Galileo-rescue:End_Sensor-Quanser_2DSFJE_Library
- U1: symbol Quanser_2DSFJE_Library:LS7366R -> Shield_Galileo-rescue:LS7366R-Quanser_2DSFJE_Library
- U2: symbol Quanser_2DSFJE_Library:Intel_Galileo_Gen2 -> Shield_Galileo-rescue:Intel_Galileo_Gen2-Quanser_2DSFJE_Library
Connections:
- net at C4.1, U3.4 (Vs): no longer J3.2 (Pin_2)
Other:
- moved on the sheet: U4G
Changed lines of the file:
@@
 Schematic for Intel® Galileo Gen2 Shield
 $Comp
-L Quanser_2DSFJE_Library:Intel_Galileo_Gen2 U2
+L Shield_Galileo-rescue:Intel_Galileo_Gen2-Quanser_2DSFJE_Library U2
 U 1 1 5DB071F2
 P 2800 4050
@@
 $EndComp
 $Comp
-L Quanser_2DSFJE_Library:LS7366R U1
+L Shield_Galileo-rescue:LS7366R-Quanser_2DSFJE_Library U1
 U 1 1 5DB0F7D8
 P 4400 1450
@@
 NoConn ~ 1650 5950
 $Comp
-L Quanser_2DSFJE_Library:End_Sensor J2
+L Shield_Galileo-rescue:End_Sensor-Quanser_2DSFJE_Library J2
 U 1 1 5DBA5CC4
 P 4800 4900
@@
 	1    0    0    -1
 $EndComp
-$Comp
-L Driver_Motor:L298HN U3
-U 1 1 5DD1FF24
-P 7800 3700
-F 0 "U3" H 7800 4581 50  0000 C CNN
-F 1 "L298HN" H 7800 4490 50  0000 C CNN
-F 2 "L298N:TO127P2020X500X2100-15" H 7850 3050 50  0001 L CNN
-F 3 "http://www.st.com/st-web-ui/static/active/en/resource/technical/document/datasheet/CD00000240.pdf" H 7950 3950 50  0001 C CNN
-	1    7800 3700
-	1    0    0    -1
-$EndComp
-Wire Wire Line
-	7900 3000 8050 3000
-Wire Wire Line
-	8050 3000 8050 2400
 Wire Wire Line
 	8350 2400 8050 2400
@@
 Wire Wire Line
 	7800 3000 7800 2950
-Connection ~ 7800 3000
 Wire Wire Line
 	9450 2950 9450 3850
-Connection ~ 8050 3000
 Wire Wire Line
 	9450 4500 9900 4500
@@
 B_J1
 $Comp
-L Quanser_2DSFJE_Library:Connector_Encoder J1
+L Shield_Galileo-rescue:Connector_Encoder-Quanser_2DSFJE_Library J1
 U 1 1 5DDA378C
 P 7000 1900
@@
 $EndComp
 Wire Wire Line
-	8050 3000 9900 3000
-Wire Wire Line
 	7800 2950 9000 2950
 Wire Wire Line
@@
 L 74xx:74HC04 U4
 U 7 1 5DEE1C35
-P 6400 5650
-F 0 "U4" H 6630 5696 50  0000 L CNN
-F 1 "74HC04" H 6630 5605 50  0000 L CNN
-F 2 "Quanser_2DSFJE_Library:DIP-14_W7.62mm" H 6400 5650 50  0001 C CNN
-F 3 "https://assets.nexperia.com/documents/data-sheet/74HC_HCT04.pdf" H 6400 5650 50  0001 C CNN
-	7    6400 5650
+P 6550 5500
+F 0 "U4" H 6780 5546 50  0000 L CNN
+F 1 "74HC04" H 6780 5455 50  0000 L CNN
+F 2 "Quanser_2DSFJE_Library:DIP-14_W7.62mm" H 6550 5500 50  0001 C CNN
+F 3 "https://assets.nexperia.com/documents/data-sheet/74HC_HCT04.pdf" H 6550 5500 50  0001 C CNN
+	7    6550 5500
 	1    0    0    -1
 $EndComp
@@
 L power:Earth #PWR013
 U 1 1 5DEE42B1
-P 6400 6150
-F 0 "#PWR013" H 6400 5900 50  0001 C CNN
-F 1 "Earth" H 6400 6000 50  0001 C CNN
-F 2 "" H 6400 6150 50  0001 C CNN
-F 3 "~" H 6400 6150 50  0001 C CNN
-	1    6400 6150
+P 6550 6000
+F 0 "#PWR013" H 6550 5750 50  0001 C CNN
+F 1 "Earth" H 6550 5850 50  0001 C CNN
+F 2 "" H 6550 6000 50  0001 C CNN
+F 3 "~" H 6550 6000 50  0001 C CNN
+	1    6550 6000
 	1    0    0    -1
 $EndComp
@@
 L power:+5V #PWR012
 U 1 1 5DEE4D6D
-P 6400 5150
-F 0 "#PWR012" H 6400 5000 50  0001 C CNN
-F 1 "+5V" H 6415 5323 50  0000 C CNN
-F 2 "" H 6400 5150 50  0001 C CNN
-F 3 "" H 6400 5150 50  0001 C CNN
-	1    6400 5150
+P 6550 5000
+F 0 "#PWR012" H 6550 4850 50  0001 C CNN
+F 1 "+5V" H 6565 5173 50  0000 C CNN
+F 2 "" H 6550 5000 50  0001 C CNN
+F 3 "" H 6550 5000 50  0001 C CNN
+	1    6550 5000
 	1    0    0    -1
 $EndComp
@@
 	1    0    0    -1
 $EndComp
+Connection ~ 7800 3000
+$Comp
+L Driver_Motor:L298HN U3
+U 1 1 5DD1FF24
+P 7800 3700
+F 0 "U3" H 7800 4581 50  0000 C CNN
+F 1 "L298HN" H 7800 4490 50  0000 C CNN
+F 2 "L298N:TO127P2020X500X2100-15" H 7850 3050 50  0001 L CNN
+F 3 "http://www.st.com/st-web-ui/static/active/en/resource/technical/document/datasheet/CD00000240.pdf" H 7950 3950 50  0001 C CNN
+	1    7800 3700
+	1    0    0    -1
+$EndComp
+Wire Wire Line
+	8050 2400 8050 3050
+Wire Wire Line
+	7900 3000 9900 3000
 $EndSCHEMATC
