File: shield/_autosave-Shield_Galileo.kicad_pcb (KiCad board)
At the start: 2 copper layers, 144.3 x 78.7 mm, 20 parts, among them J1 Connector_Encoder, J2 End_Sensor, J3 27V Power Supply, J4 Motor, U1 LS7366R, U2 Intel_Galileo_Gen2, U3 L298HN, U4 74HC04, Y1 32MHz

Commit message: Add new Shield files
Routing:
- net /!PWM: track 43.0 -> 48.4 mm
- net /!(!PWM): track 26.2 -> 28.7 mm
- net Net-(D2-Pad1): track 120.0 -> 120.7 mm
